File: PCB/detector/detector.sch (EAGLE design)
At the start: 36 parts, among them IC1 STM32F042K6T6

Commit message: almost ready
Parts:
- removed +3.3V, +5V: (no value), con-ptr500:AK500/2
- removed D1: 3.3V, diode:ZENER-DIODESOD80C
- removed JP1: (no value), pinhead:PINHD-1X3/90
- removed JP2: (no value), pinhead:PINHD-1X4/90
- removed Q1: (no value), crystal:CRYSTALCTS406
- removed S1: DTSM-3, swtich:DTSM-3
- added BAT1: BAT_3V, battery CR1216:BAT_3V
- added C18, C23: 100nF, resistor:C-EUC0603
- added C19, C20, C21, C22: 22pF, resistor:C-EUC0603
- added C24: 1u, rcl:C-EUC0603
- added C25: 100p, rcl:C-EUC0603
- added C26: 100n, rcl:C-EUC0603
- added C27, C28: 1n, rcl:C-EUC0603
- added CAN+PWR: 4PIN_3.81_KATOWA, zielone raster 3.81:4PIN_3.81_KATOWA
- added CR1: 32,768kHz, crystal_scorpio:IL3X
- added D3_SK1: 5A, diode:DIODE-DO214AA
- added DA1: SN65HVD230, can_driver:SN65HVD230
- added FUSE1: 3A, resistor:R-EU_R0603
- added L1: 1uH/500mA, rcl:L-USL2012C
- added L2: 10uH/20mA, rcl:L-USL2012C
- added L3, L4: (no value), rcl:L-EUL3216C
- added LED1, LED3: zielona, led:LEDCHIP-LED0603
- added LED2: niebieska, led:LEDCHIP-LED0603
- added LED4: czerwona, led:LEDCHIP-LED0603
- added MA_BYC_ACS711_!!: ACS712, acs712:ACS712
- added PROGRAMATOR: (no value), pinhead:PINHD-1X6
- added PRZETWORNICA1: 3.3V, OKI-78SR:OKI78-SR
- added R10: 120R*, resistor:R-EU_R0603
- added R11: 390k, resistor:R-EU_R0603
- added R12, R13: 10k, resistor:R-EU_R0603
- added R14, R15, R16: 470R, resistor:R-EU_R0603
- added TRANSIL1: 3.3V, diode:SUPPRESSOR-SMBJ
- added U$2: STM32F072RBT6, STM32F072RBT6:STM32F072RBT6
- added U$3: ABM3, crystal_scorpio:ABM3
- added U$6: LC03-6R2G, LC03-6R2 - diody ESD do magistrali:LC03-6R2G
- added U1: LT5538, DFN-8:LT5538
- added U2: B39431B3710U410, SON120P300X300X110-6N:B39431B3710U410
- added ZW_MASY: (no value), resistor:R-EU_R0603
- added ZW_ZASILANIA: (no value), pinhead:PINHD-1X2
- C1: value 100n -> (none); device rcl:C-EUC0805 -> rcl:C-EUC0603
- C10, C12, C15: value 100n -> 100nF; device rcl:C-EUC0805 -> resistor:C-EUC0603
- C11, C9: value 4.7u -> 100nF; device rcl:CPOL-EUCT3216 -> resistor:C-EUC0603
- C13: value 10n -> 100nF; device rcl:C-EUC0805 -> resistor:C-EUC0603
- C14: value 1u -> 100nF; device rcl:CPOL-EUCT3216 -> resistor:C-EUC0603
- C16: value 20p -> 100nF; device rcl:C-EUC0805 -> resistor:C-EUC0603
- C17: value 20p -> 6,3V/100uF; device rcl:C-EUC0805 -> resistor:CPOL-EUE2-5
- C2: value 100p -> 4,7uF; device rcl:C-EUC0805 -> rcl:CPOL-EUSMCA
- C3: value 100p -> (none); device rcl:C-EUC0805 -> rcl:C-EUC0603
- C4: device rcl:C-EUC0805 -> rcl:C-EUC0603
- C5, C6: value 100n -> 100p; device rcl:C-EUC0805 -> rcl:C-EUC0603
- C7: value 10u -> 4,7uF; device rcl:C-EUC0805 -> rcl:CPOL-EUSMCA
- C8: value 100n -> 1uF; device rcl:C-EUC0805 -> resistor:C-EUC0603
- IC1: value STM32F042K6T6 -> LM50; device STM32F042K6T6:STM32F042K6T6 -> linear:LM50
- R1: value 60.4R -> VARISTORCN0603; device rcl:R-EU_R0805 -> varistor:VARISTORCN0603
- R2: value 2k -> (none); device rcl:R-EU_R0805 -> rcl:R-EU_R0603
- R3: value 301R -> 820R; device rcl:R-EU_R0805 -> resistor:R-EU_R0603
- R4: value 10k -> 56R; device rcl:R-EU_R0805 -> rcl:R-EU_R0603
- R5: value 20k -> (none); device rcl:R-EU_R0805 -> rcl:R-EU_R0603
- R6: value 1430R -> 10k; device rcl:R-EU_R0805 -> resistor:R-EU_R0603
- R7: value 3.74k -> 100K; device rcl:R-EU_R0805 -> resistor:R-EU_R0603
- R8: value 2k -> ZW 0-100K; device rcl:R-EU_R0805 -> resistor:R-EU_R0603
- R9: value 0R -> 32k; device rcl:R-EU_R0805 -> resistor:R-EU_R0603
- U$1: value ADL5902 -> TQP3M9036; device ADL5902:ADL5902 -> DFN-8:TQP3M9036
Connections:
- net N$1 renamed SIGNAL
- removed net +5V: +5V-1.KL, C3.1, C4.1, C5.1, C6.1, U$1.VPOS1, U$1.VPOS2
- removed net ADC_IN: D1.C, IC1.PA0, R2.1
- removed net INHI: C1.2, U$1.INHI
- removed net OSC_IN: C17.1, IC1.PF0, Q1.2
- removed net OSC_OUT: C16.1, IC1.PF1, Q1.1
- removed net RESET: C15.1, IC1.!RST, JP2.2, S1.1
- removed net SWCLK: IC1.PA14, JP2.3
- removed net UART_RX: IC1.PA10, JP1.2
- removed net UART_TX: IC1.PA9, JP1.3
- removed net VOUT: R4.2, R9.2, U$1.VOUT
- new net +24V: C14.1, D3_SK1.C, PRZETWORNICA1.P$1
- new net AGND: C18.2, C7.-, C8.2, C9.2, IC1.GND, MA_BYC_ACS711_!!.GND, R9.1, U$2.VSSA, ZW_MASY.2
- new net AMP_OUT: C27.2, C5.2, R4.2
- new net BOOT_0: PROGRAMATOR.4, R12.2, U$2.BOOT0
- new net CANH_1: DA1.CANH, R10.2, U$6.IN_1
- new net CANL_1: DA1.CANL, R10.1, U$6.IN_2
- new net CAN_RX_1: DA1.RXD, U$2.PB8
- new net CAN_TX_1: DA1.TXD, U$2.PB9
- new net DET_OUT: R5.2, U$2.PA3
- new net FILTER_IN: C3.2, U2.IN
- new net FILTER_OUT: C4.1, U2.OUT
- new net LED1: LED3.A, U$2.PC3
- new net LED2: LED4.A, U$2.PA2
- new net N$1: MA_BYC_ACS711_!!.VOUT, R7.1
- new net N$10: C19.1, U$2.PF0-OSC_IN, U$3.P$1
- new net N$11: C4.2, U$1.IN
- new net N$12: CAN+PWR.P2, U$6.OUT_1
- new net N$13: R11.1, U$2.PC15-OSC32_OUT
- new net N$14: C21.1, CR1.P$1, U$2.PC14-OSC32_IN
- new net N$15: C22.1, CR1.P$2, R11.2
- new net N$16: CAN+PWR.P1, U$6.OUT_2
- new net N$18: LED1.A, R13.1
- new net N$19: LED2.A, R14.1
- new net N$20: LED3.C, R15.2
- new net N$21: LED4.C, R16.2
- new net N$22: C28.1, U1.IN-
- new net N$23: C27.1, U1.IN+
- new net N$24: PROGRAMATOR.2, ZW_ZASILANIA.1
- new net N$25: R2.2, U1.ENBL
- new net N$27: C5.1, L4.2, U$1.OUT
- new net N$28: U1.CAP+
- new net N$29: U1.CAP-
- new net N$8: D3_SK1.A, MA_BYC_ACS711_!!.I+_0, MA_BYC_ACS711_!!.I+_1
- new net NRST: C23.1, PROGRAMATOR.3, U$2.NRST
- new net OVER_CURRENT: MA_BYC_ACS711_!!.FILTER, R6.2, U$2.PC13
- new net PRAD_PLYTKI: R7.2, R9.2, U$2.PC0
- new net SWD_CLK: PROGRAMATOR.5, U$2.PA14
- new net TEMP: IC1.VO, U$2.PC1
- new net VBAT: BAT1.P$1+, U$2.VBAT
- new net VCC: CAN+PWR.P4, MA_BYC_ACS711_!!.I-_0, MA_BYC_ACS711_!!.I-_1, R13.2
- new net VDD: C10.1, C11.1, C12.1, C13.1, C15.2, C18.1, C2.+, DA1.VDD, IC1.+VS, L1.1, L2.1, MA_BYC_ACS711_!!.VCC, R6.1, U$2.VDD1, U$2.VDD2, U$2.VDD3, U$2.VDDIO2, ZW_ZASILANIA.2
- net +3V3: now also C24.1, C25.1, C26.1, C6.1, FUSE1.2, L1.2, L4.1, R14.2, R2.1, TRANSIL1.C, U1.VCC; no longer +3.3V-1.KL, C10.1, C11.+, C12.1, C13.1, C14.+, C8.1, C9.+, IC1.VDD, IC1.VDDA, IC1.VDDIO2
- net GND: now also BAT1.P$2-, C11.2, C14.2, C15.1, C17.-, C19.2, C2.-, C20.2, C21.2, C22.2, C23.2, C24.2, C25.2, C26.2, C28.2, CAN+PWR.P3, DA1.VSS, L3.2, LED1.C, LED2.C, PROGRAMATOR.1, PRZETWORNICA1.P$2, R12.1, R15.1, R16.1, R4.1, R8.2, TRANSIL1.A, U$1.GND, U$1.NC1, U$1.NC2, U$1.NC3, U$1.NC4, U$1.NC5, U$2.VSS1, U$2.VSS2, U$2.VSS3, U$2.VSS4, U$3.P$2, U$6.NC_1, U$6.NC_2, U$6.NC_3, U$6.NC_4, U1.GND, U1.P_GND, U2.GND, U2.GND2, U2.GND3, U2.GND4, ZW_MASY.1; no longer +3.3V-2.KL, +5V-2.KL, C11.-, C14.-, C15.2, C17.2, C2.2, C3.2, C4.2, C5.2, C7.2, C8.2, C9.-, D1.A, IC1.VSS, IC1.VSSA, JP1.1, JP2.1, R3.1, R5.1, R8.1, S1.2, U$1.COMM1, U$1.COMM2
- net N$2: now also C16.1, C17.+, FUSE1.1, PRZETWORNICA1.P$3; no longer R6.2, R7.2, U$1.VREF
- net N$3: now also R3.1, U$2.PF1-OSC_OUT; no longer C2.1, U$1.INLO
- net N$4: now also C7.+, C8.1, C9.1, L2.2, U$2.VDDA; no longer C7.1, U$1.CLPF
- net N$5: now also C1.2, C3.1, L3.1; no longer R2.2, R4.1, R5.2
- net N$6: now also C20.1, R3.2, U$3.P$3; no longer R9.1, U$1.VSET
- net N$7: now also DA1.RS, R8.1; no longer R3.2, R6.1, U$1.TADJ/PWDN
- net N$9: now also R5.1, U1.VOUT; no longer R7.1, R8.2, U$1.VTGT
- net SWDIO: now also PROGRAMATOR.6, U$2.PA13; no longer IC1.PA13, JP2.4
Other:
- note added: "AMPLIFIER"
- note added: "Do procesora"
- note added: "FILTER"
- note removed: "CONVERTER"

Commit message: rf circut edited, pololu lbr added
Parts:
- removed BAT1: BAT_3V, battery CR1216:BAT_3V
- removed C10, C11, C12, C13, C14, C15, C16, C18, C23: 100nF, resistor:C-EUC0603
- removed C17: 6,3V/100uF, resistor:CPOL-EUE2-5
- removed C19, C20, C21, C22: 22pF, resistor:C-EUC0603
- removed C25: 100p, rcl:C-EUC0603
- removed C26: 100n, rcl:C-EUC0603
- removed C27, C28: 1n, rcl:C-EUC0603
- removed CAN+PWR: 4PIN_3.81_KATOWA, zielone raster 3.81:4PIN_3.81_KATOWA
- removed CR1: 32,768kHz, crystal_scorpio:IL3X
- removed D3_SK1: 5A, diode:DIODE-DO214AA
- removed DA1: SN65HVD230, can_driver:SN65HVD230
- removed FUSE1: 3A, resistor:R-EU_R0603
- removed IC1: LM50, linear:LM50
- removed L1: 1uH/500mA, rcl:L-USL2012C
- removed L2: 10uH/20mA, rcl:L-USL2012C
- removed LED1, LED3: zielona, led:LEDCHIP-LED0603
- removed LED2: niebieska, led:LEDCHIP-LED0603
- removed LED4: czerwona, led:LEDCHIP-LED0603
- removed MA_BYC_ACS711_!!: ACS712, acs712:ACS712
- removed PROGRAMATOR: (no value), pinhead:PINHD-1X6
- removed PRZETWORNICA1: 3.3V, OKI-78SR:OKI78-SR
- removed R10: 120R*, resistor:R-EU_R0603
- removed R11: 390k, resistor:R-EU_R0603
- removed R12, R13: 10k, resistor:R-EU_R0603
- removed R14, R15, R16: 470R, resistor:R-EU_R0603
- removed R2, R5: (no value), rcl:R-EU_R0603
- removed R4: 56R, rcl:R-EU_R0603
- removed R8: ZW 0-100K, resistor:R-EU_R0603
- removed R9: 32k, resistor:R-EU_R0603
- removed TRANSIL1: 3.3V, diode:SUPPRESSOR-SMBJ
- removed U$2: STM32F072RBT6, STM32F072RBT6:STM32F072RBT6
- removed U$3: ABM3, crystal_scorpio:ABM3
- removed U$6: LC03-6R2G, LC03-6R2 - diody ESD do magistrali:LC03-6R2G
- removed U1: LT5538, DFN-8:LT5538
- removed ZW_MASY: (no value), resistor:R-EU_R0603
- removed ZW_ZASILANIA: (no value), pinhead:PINHD-1X2
- added U3: LT5537EDDBTRPBF, LT5537EDDBTRPBF:LT5537EDDBTRPBF
- C2, C7: value 4,7uF -> 100p; device rcl:CPOL-EUSMCA -> rcl:C-EUC0603
- C8: value 1uF -> 1n; device resistor:C-EUC0603 -> rcl:C-EUC0603
- C9: value 100nF -> 1u; device resistor:C-EUC0603 -> rcl:C-EUC0603
- R3: value 820R -> (none); device resistor:R-EU_R0603 -> rcl:R-EU_R0603
- R6: value 10k -> 51R; device resistor:R-EU_R0603 -> rcl:R-EU_R0603
- R7: value 100K -> 33k; device resistor:R-EU_R0603 -> rcl:R-EU_R0603
Connections:
- removed net +24V: C14.1, D3_SK1.C, PRZETWORNICA1.P$1
- removed net AGND: C18.2, C7.-, C8.2, C9.2, IC1.GND, MA_BYC_ACS711_!!.GND, R9.1, U$2.VSSA, ZW_MASY.2
- removed net BOOT_0: PROGRAMATOR.4, R12.2, U$2.BOOT0
- removed net CANH_1: DA1.CANH, R10.2, U$6.IN_1
- removed net CANL_1: DA1.CANL, R10.1, U$6.IN_2
- removed net CAN_RX_1: DA1.RXD, U$2.PB8
- removed net CAN_TX_1: DA1.TXD, U$2.PB9
- removed net LED1: LED3.A, U$2.PC3
- removed net LED2: LED4.A, U$2.PA2
- removed net N$10: C19.1, U$2.PF0-OSC_IN, U$3.P$1
- removed net N$12: CAN+PWR.P2, U$6.OUT_1
- removed net N$13: R11.1, U$2.PC15-OSC32_OUT
- removed net N$14: C21.1, CR1.P$1, U$2.PC14-OSC32_IN
- removed net N$15: C22.1, CR1.P$2, R11.2
- removed net N$16: CAN+PWR.P1, U$6.OUT_2
- removed net N$18: LED1.A, R13.1
- removed net N$19: LED2.A, R14.1
- removed net N$20: LED3.C, R15.2
- removed net N$21: LED4.C, R16.2
- removed net N$22: C28.1, U1.IN-
- removed net N$23: C27.1, U1.IN+
- removed net N$24: PROGRAMATOR.2, ZW_ZASILANIA.1
- removed net N$25: R2.2, U1.ENBL
- removed net N$28: U1.CAP+
- removed net N$29: U1.CAP-
- removed net N$4: C7.+, C8.1, C9.1, L2.2, U$2.VDDA
- removed net N$6: C20.1, R3.2, U$3.P$3
- removed net N$7: DA1.RS, R8.1
- removed net N$8: D3_SK1.A, MA_BYC_ACS711_!!.I+_0, MA_BYC_ACS711_!!.I+_1
- removed net N$9: R5.1, U1.VOUT
- removed net NRST: C23.1, PROGRAMATOR.3, U$2.NRST
- removed net OVER_CURRENT: MA_BYC_ACS711_!!.FILTER, R6.2, U$2.PC13
- removed net PRAD_PLYTKI: R7.2, R9.2, U$2.PC0
- removed net SWDIO: PROGRAMATOR.6, U$2.PA13
- removed net SWD_CLK: PROGRAMATOR.5, U$2.PA14
- removed net TEMP: IC1.VO, U$2.PC1
- removed net VBAT: BAT1.P$1+, U$2.VBAT
- removed net VCC: CAN+PWR.P4, MA_BYC_ACS711_!!.I-_0, MA_BYC_ACS711_!!.I-_1, R13.2
- removed net VDD: C10.1, C11.1, C12.1, C13.1, C15.2, C18.1, C2.+, DA1.VDD, IC1.+VS, L1.1, L2.1, MA_BYC_ACS711_!!.VCC, R6.1, U$2.VDD1, U$2.VDD2, U$2.VDD3, U$2.VDDIO2, ZW_ZASILANIA.2
- net +3V3: now also C8.1, C9.1, R3.1, U3.VCC; no longer C25.1, C26.1, FUSE1.2, L1.2, R14.2, R2.1, TRANSIL1.C, U1.VCC
- net AMP_OUT: now also C2.2, R6.2; no longer C27.2, R4.2
- net DET_OUT: now also R7.1, U3.OUT; no longer R5.2, U$2.PA3
- net GND: now also C7.2, C8.2, C9.2, R6.1, R7.2, U3.CAP+, U3.CAP-, U3.EPAD, U3.VEE; no longer BAT1.P$2-, C10.2, C11.2, C12.2, C13.2, C14.2, C15.1, C16.2, C17.-, C19.2, C2.-, C20.2, C21.2, C22.2, C23.2, C25.2, C26.2, C28.2, CAN+PWR.P3, DA1.VSS, LED1.C, LED2.C, PROGRAMATOR.1, PRZETWORNICA1.P$2, R12.1, R15.1, R16.1, R4.1, R8.2, TRANSIL1.A, U$2.VSS1, U$2.VSS2, U$2.VSS3, U$2.VSS4, U$3.P$2, U$6.NC_1, U$6.NC_2, U$6.NC_3, U$6.NC_4, U1.GND, U1.P_GND, ZW_MASY.1
- net N$1: now also R3.2, U3.ENBL; no longer MA_BYC_ACS711_!!.VOUT, R7.1
- net N$2: now also C7.1, U3.IN-; no longer C16.1, C17.+, FUSE1.1, PRZETWORNICA1.P$3
- net N$3: now also C2.1, U3.IN+; no longer R3.1, U$2.PF1-OSC_OUT
Other:
- note removed: "Do procesora"

Commit message: reinstall
Parts:
- L3, L4: device rcl:L-EUL3216C -> rcl:L-EUL2012C
Changed lines of the file:
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@@
 <part name="GND4" library="supply1" library_urn="urn:adsk.eagle:library:371" deviceset="GND" device=""/>
 <part name="R1" library="varistor" library_urn="urn:adsk.eagle:library:410" deviceset="VARISTOR" device="CN0603" package3d_urn="urn:adsk.eagle:package:30597/1"/>
-<part name="L3" library="rcl" library_urn="urn:adsk.eagle:library:334" deviceset="L-EU" device="L3216C" package3d_urn="urn:adsk.eagle:package:23476/2"/>
+<part name="L3" library="rcl" library_urn="urn:adsk.eagle:library:334" deviceset="L-EU" device="L2012C" package3d_urn="urn:adsk.eagle:package:23475/1"/>
 <part name="C1" library="rcl" library_urn="urn:adsk.eagle:library:334" deviceset="C-EU" device="C0603" package3d_urn="urn:adsk.eagle:package:23616/2"/>
 <part name="C3" library="rcl" library_urn="urn:adsk.eagle:library:334" deviceset="C-EU" device="C0603" package3d_urn="urn:adsk.eagle:package:23616/2"/>
@@
 <part name="C6" library="rcl" library_urn="urn:adsk.eagle:library:334" deviceset="C-EU" device="C0603" package3d_urn="urn:adsk.eagle:package:23616/2" value="100p"/>
 <part name="C24" library="rcl" library_urn="urn:adsk.eagle:library:334" deviceset="C-EU" device="C0603" package3d_urn="urn:adsk.eagle:package:23616/2" value="1u"/>
-<part name="L4" library="rcl" library_urn="urn:adsk.eagle:library:334" deviceset="L-EU" device="L3216C" package3d_urn="urn:adsk.eagle:package:23476/2"/>
+<part name="L4" library="rcl" library_urn="urn:adsk.eagle:library:334" deviceset="L-EU" device="L2012C" package3d_urn="urn:adsk.eagle:package:23475/1"/>
 <part name="GND31" library="supply1" library_urn="urn:adsk.eagle:library:371" deviceset="GND" device=""/>
 <part name="+3V1" library="supply1" library_urn="urn:adsk.eagle:library:371" deviceset="+3V3" device=""/>

Commit message: first connection commit
Parts:
- added C10, C11, C12, C13, C14, C15, C18, C22: 100nF, resistor:C-EUC0603
- added C16: 1uF, resistor:C-EUC0603
- added C17, C19: 4,7uF, rcl:CPOL-EUSMCA
- added C20, C21: 22pF, resistor:C-EUC0603
- added CAN+PWR: 4PIN_3.81_KATOWA, zielone raster 3.81:4PIN_3.81_KATOWA
- added DA1: SN65HVD230, can_driver:SN65HVD230
- added FUSE1: 3A, resistor:R-EU_R0603
- added IC1: LM50, linear:LM50
- added L1: 1uH/500mA, rcl:L-USL2012C
- added L2: 10uH/20mA, rcl:L-USL2012C
- added LED1: zielona, led:LEDCHIP-LED0603
- added LED2: niebieska, led:LEDCHIP-LED0603
- added MA_BYC_ACS711_!!: ACS712, acs712:ACS712
- added PROGRAMATOR: (no value), pinhead:PINHD-1X6
- added Q1: (no value), transistor-power:P-MOSFET-SO8
- added R10: ZW 0-100K, resistor:R-EU_R0603
- added R11: 120R*, resistor:R-EU_R0603
- added R12, R14, R15: 10k, resistor:R-EU_R0603
- added R13: 820R, resistor:R-EU_R0603
- added R16: 470R, resistor:R-EU_R0603
- added R17, R9: 32k, resistor:R-EU_R0603
- added R2, R4, R5: (no value), rcl:R-EU_R0603
- added R8: 100K, resistor:R-EU_R0603
- added SIGNAL1: (no value), adafruit:SMACONNECTOR_EDGE
- added TRANSIL1: 3.3V, diode:SUPPRESSOR-SMBJ
- added U$2: STM32F072RBT6, STM32F072RBT6:STM32F072RBT6
- added U$3: ABM3, crystal_scorpio:ABM3
- added U$4: D24V22F3, przetwornice:D24V22F3
- added U$6: LC03-6R2G, LC03-6R2 - diody ESD do magistrali:LC03-6R2G
- added ZW_MASY: (no value), resistor:R-EU_R0603
- added ZW_ZASILANIA: (no value), pinhead:PINHD-1X2
Connections:
- new net +24V: Q1.S, R15.2, U$4.IN+
- new net AGND: C14.2, C16.2, C17.-, C18.2, IC1.GND, MA_BYC_ACS711_!!.GND, R9.1, U$2.VSSA, ZW_MASY.2
- new net BOOT_0: PROGRAMATOR.4, R14.2, U$2.BOOT0
- new net CANH_1: DA1.CANH, R11.2, U$6.IN_1
- new net CANL_1: DA1.CANL, R11.1, U$6.IN_2
- new net CAN_RX_1: DA1.RXD, U$2.PB8
- new net CAN_TX_1: DA1.TXD, U$2.PB9
- new net LED1_ON: U$2.PA1
- new net LED2_ON: U$2.PA2
- new net LED3_ON: U$2.PA3
- new net N$10: MA_BYC_ACS711_!!.I+_0, MA_BYC_ACS711_!!.I+_1, Q1.D
- new net N$12: R13.1, U$2.PF1-OSC_OUT
- new net N$13: C20.1, U$2.PF0-OSC_IN, U$3.P$1
- new net N$14: C14.1, C16.1, C17.+, L2.2, U$2.VDDA
- new net N$15: C21.1, R13.2, U$3.P$3
- new net N$16: CAN+PWR.P2, U$6.OUT_1
- new net N$17: CAN+PWR.P1, U$6.OUT_2
- new net N$18: LED1.A, R15.1
- new net N$19: LED2.A, R16.1
- new net N$20: Q1.G, R17.1
- new net N$24: PROGRAMATOR.2, ZW_ZASILANIA.1
- new net N$4: R2.1, SIGNAL.ANT
- new net N$6: R4.1, SIGNAL1.ANT
- new net N$7: MA_BYC_ACS711_!!.VOUT, R8.1
- new net N$8: DA1.RS, R10.1
- new net N$9: FUSE1.1, U$4.OUT+
- new net NRST: C22.1, PROGRAMATOR.3, U$2.NRST
- new net OVER_CURRENT: MA_BYC_ACS711_!!.FILTER, R12.2, U$2.PC13
- new net PRAD_PLYTKI: R8.2, R9.2, U$2.PC0
- new net SIGNAL1: R2.2, R4.2, R5.2
- new net SWDIO: PROGRAMATOR.6, U$2.PA13
- new net SWD_CLK: PROGRAMATOR.5, U$2.PA14
- new net TEMP: IC1.VO, U$2.PC1
- new net VCC: CAN+PWR.P4, MA_BYC_ACS711_!!.I-_0, MA_BYC_ACS711_!!.I-_1
- new net VDD: C10.1, C11.1, C12.1, C13.1, C15.2, C18.1, C19.+, DA1.VDD, IC1.+VS, L1.1, L2.1, MA_BYC_ACS711_!!.VCC, R12.1, U$2.VDD1, U$2.VDD2, U$2.VDD3, U$2.VDDIO2, ZW_ZASILANIA.2
- net +3V3: now also FUSE1.2, L1.2, R16.2, TRANSIL1.C
- net GND: now also C10.2, C11.2, C12.2, C13.2, C15.1, C19.-, C20.2, C21.2, C22.2, CAN+PWR.P3, DA1.VSS, LED1.C, LED2.C, PROGRAMATOR.1, R10.2, R14.1, R17.2, SIGNAL1.GND1, SIGNAL1.GND2, SIGNAL1.GND3, SIGNAL1.GND4, TRANSIL1.A, U$2.VSS1, U$2.VSS2, U$2.VSS3, U$2.VSS4, U$3.P$2, U$4.IN-, U$4.OUT-, U$6.NC_1, U$6.NC_2, U$6.NC_3, U$6.NC_4, ZW_MASY.1
- net SIGNAL: now also R5.1; no longer SIGNAL.ANT
Other:
- note added: "Do procesora"

Commit message: imu added
Parts:
- added C23: 10nF, resistor:C-EUC0603
- added C25, C26, C27: 100nF, resistor:C-EUC0603
- added C28, C29: 10uF, resistor:CPOL-EUSMCA
- added L5: 10uH, resistor:L-USL2012C
- added R18: 100R, resistor:R-EU_R0603
- added U$5: LSM9DS1TR, LSM9DS1TR akcelerometr, żyroskop, magnetometr:LSM9DS1TR
Connections:
- removed net DET_OUT: R7.1, U3.OUT
- new net CS_AG: U$2.PC6, U$5.CS_A/G
- new net CS_M: U$2.PC7, U$5.CS_M
- new net DEN_AG: U$5.DEN_A/G
- new net DET_ADC: R7.1, U$2.PA4, U3.OUT
- new net DRDY_M: U$5.DRDY_M
- new net INT1_AG: U$5.INT1_A/G
- new net INT2_AG: U$5.INT2_A/G
- new net INT_M: U$5.INT_M
- new net N$21: C27.1, C28.+, R18.2, U$5.VDD@1, U$5.VDD@2
- new net N$22: C23.1, U$5.CAP
- new net N$23: C26.1, U$5.C1
- new net N$25: C25.2, C29.+, L5.2, R18.1, U$5.VDD_IO, U$5.VDD_IO_1
- new net SCK: U$2.PB13, U$5.SCL/SPC
- new net SDI: U$2.PB14, U$5.SDA/SDI/SDO
- new net SDO: U$2.PB15, U$5.SDO_A/G, U$5.SDO_M
- net +3V3: now also L5.1
- net GND: now also C23.2, C25.1, C26.2, C27.2, C28.-, C29.-, U$5.GND@1, U$5.GND@2, U$5.RES@1, U$5.RES@2, U$5.RES@3, U$5.RES@4, U$5.RES@5
